File: schematics/src/ioboard/ioboard.brd (EAGLE design)
At the start: 43.2 x 99.1 mm, 34 parts, among them IC3 TL071P

Commit message: Fixed issues
Parts:
- removed R51: 10M, resistor:0207/7
- R49: value 120K -> 91k
Connections:
- removed net N$38: IC3.2, R31.1, R34.1, R49.2, R51.1
- net +12V: now also IC3.2, R31.1, R34.1, R49.2; no longer R51.2
Routing:
- net N$38: track 35.2 -> 0.00 mm
- net +12V: track 102.2 -> 122.9 mm
Other:
- board text added: "CURTIS 3340 VCO v1.2 2022 GERBSTER.NL"
- board text removed: "CURTIS 3340 VCO v1.1 2020 GERBSTER.NL"
Changed lines of the file:
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@@
 <hole x="8.255" y="81.915" drill="3.2004"/>
 <circle x="8.255" y="81.915" radius="2.9972" width="0.1524" layer="25"/>
-<text x="33.02" y="72.39" size="1.6764" layer="25" font="vector" rot="R90">CURTIS 3340 VCO v1.1
-2020 GERBSTER.NL</text>
+<text x="33.02" y="72.39" size="1.6764" layer="25" font="vector" rot="R90">CURTIS 3340 VCO v1.2
+2022 GERBSTER.NL</text>
 </plain>
 <attributes>
@@
 <attribute name="VALUE" x="13.0556" y="32.2326" size="0.9906" layer="27" ratio="10" rot="R180"/>
 </element>
-<element name="R49" library="resistor" package="0207/7" value="120K" x="21.59" y="31.75" smashed="yes" rot="R180">
+<element name="R49" library="resistor" package="0207/7" value="91k" x="21.59" y="31.75" smashed="yes" rot="R180">
 <attribute name="NAME" x="24.13" y="32.385" size="0.9906" layer="25" font="vector" rot="R180"/>
 <attribute name="VALUE" x="23.2156" y="32.2326" size="0.9906" layer="27" ratio="10" rot="R180"/>
@@
 <attribute name="NAME" x="33.655" y="8.255" size="0.9906" layer="25" font="vector" rot="R180"/>
 <attribute name="VALUE" x="29.4894" y="7.1374" size="0.9906" layer="27" ratio="10"/>
-</element>
-<element name="R51" library="resistor" package="0207/7" value="10M" x="31.115" y="24.13" smashed="yes">
-<attribute name="NAME" x="33.655" y="24.765" size="0.9906" layer="25" font="vector" rot="R180"/>
-<attribute name="VALUE" x="29.4894" y="23.6474" size="0.9906" layer="27" ratio="10"/>
 </element>
 <element name="R53" library="resistor" package="0207/7" value="5.6K" x="24.765" y="14.605" smashed="yes" rot="R90">
@@
 <contactref element="JP4" pad="6"/>
 <contactref element="IC3" pad="7"/>
-<contactref element="R51" pad="2"/>
-<wire x1="33.02" y1="10.795" x2="33.02" y2="13.97" width="0.4064" layer="16"/>
-<wire x1="33.02" y1="13.97" x2="34.29" y2="15.24" width="0.4064" layer="16"/>
-<wire x1="34.29" y1="15.24" x2="34.29" y2="23.495" width="0.4064" layer="16"/>
-<wire x1="34.29" y1="23.495" x2="34.925" y2="24.13" width="0.4064" layer="16"/>
+<wire x1="33.02" y1="10.795" x2="33.02" y2="18.415" width="0.4064" layer="16"/>
 <wire x1="33.02" y1="10.795" x2="34.29" y2="9.525" width="0.4064" layer="1"/>
 <wire x1="35.56" y1="9.525" x2="37.465" y2="7.62" width="0.4064" layer="1"/>
@@
 <wire x1="24.13" y1="70.485" x2="24.13" y2="67.945" width="0.4064" layer="16"/>
 <wire x1="24.13" y1="67.93" x2="24.09" y2="67.93" width="0.4064" layer="1"/>
-<wire x1="34.925" y1="24.13" x2="36.195" y2="25.4" width="0.4064" layer="1"/>
-<wire x1="36.195" y1="27.94" x2="32.385" y2="31.75" width="0.4064" layer="1"/>
+<wire x1="34.925" y1="29.21" x2="32.385" y2="31.75" width="0.4064" layer="1"/>
 <wire x1="32.385" y1="31.75" x2="32.385" y2="65.405" width="0.4064" layer="1"/>
 <wire x1="32.385" y1="65.405" x2="29.845" y2="67.945" width="0.4064" layer="1"/>
 <wire x1="29.845" y1="67.945" x2="24.13" y2="67.945" width="0.4064" layer="1"/>
 <wire x1="24.13" y1="67.945" x2="24.13" y2="67.93" width="0.4064" layer="1"/>
-<wire x1="36.195" y1="25.4" x2="36.195" y2="27.94" width="0.4064" layer="1"/>
+<wire x1="34.925" y1="26.67" x2="34.925" y2="29.21" width="0.4064" layer="1"/>
 <via x="24.13" y="67.945" extent="1-16" drill="0.35"/>
+<contactref element="R31" pad="1"/>
+<contactref element="IC3" pad="2"/>
+<contactref element="R49" pad="2"/>
+<contactref element="R34" pad="1"/>
+<wire x1="17.78" y1="31.75" x2="15.24" y2="31.75" width="0.4064" layer="16"/>
+<wire x1="30.48" y1="26.67" x2="33.02" y2="26.67" width="0.4064" layer="1"/>
+<wire x1="33.02" y1="26.67" x2="34.925" y2="26.67" width="0.4064" layer="1"/>
+<wire x1="33.02" y1="18.415" x2="33.02" y2="26.67" width="0.4064" layer="1"/>
+<wire x1="30.48" y1="26.67" x2="27.94" y2="29.21" width="0.4064" layer="1"/>
+<wire x1="27.94" y1="29.21" x2="19.05" y2="29.21" width="0.4064" layer="1"/>
+<wire x1="19.05" y1="29.21" x2="17.78" y2="30.48" width="0.4064" layer="1"/>
+<wire x1="17.78" y1="30.48" x2="17.78" y2="31.75" width="0.4064" layer="1"/>
 </signal>
 <signal name="-12V">
@@
 <wire x1="17.78" y1="16.495" x2="17.78" y2="24.13" width="0.4064" layer="1"/>
 </signal>
-<signal name="N$38">
-<contactref element="R31" pad="1"/>
-<contactref element="IC3" pad="2"/>
-<contactref element="R49" pad="2"/>
-<contactref element="R34" pad="1"/>
-<contactref element="R51" pad="1"/>
-<wire x1="17.78" y1="31.75" x2="15.24" y2="31.75" width="0.4064" layer="16"/>
-<wire x1="27.305" y1="24.13" x2="29.21" y2="24.13" width="0.4064" layer="1"/>
-<wire x1="29.21" y1="24.13" x2="33.02" y2="24.13" width="0.4064" layer="1"/>
-<wire x1="33.02" y1="24.13" x2="33.02" y2="25.4" width="0.4064" layer="1"/>
-<wire x1="33.02" y1="25.4" x2="34.29" y2="26.67" width="0.4064" layer="1"/>
-<wire x1="34.29" y1="26.67" x2="34.925" y2="26.67" width="0.4064" layer="1"/>
-<wire x1="33.02" y1="18.415" x2="33.02" y2="24.13" width="0.4064" layer="1"/>
-<wire x1="29.21" y1="27.94" x2="27.94" y2="29.21" width="0.4064" layer="1"/>
-<wire x1="27.94" y1="29.21" x2="19.05" y2="29.21" width="0.4064" layer="1"/>
-<wire x1="19.05" y1="29.21" x2="17.78" y2="30.48" width="0.4064" layer="1"/>
-<wire x1="17.78" y1="30.48" x2="17.78" y2="31.75" width="0.4064" layer="1"/>
-<wire x1="29.21" y1="24.13" x2="29.21" y2="27.94" width="0.4064" layer="1"/>
-</signal>
 <signal name="PWM_IN_IO">
