File: schematics/src/ioboard/ioboard.sch (EAGLE design)
At the start: 34 parts, among them IC3 TL071P

Commit message: Fixed issues
Parts:
- removed R51: 10M, resistor:R-US_0207/7
- R49: value 120K -> 91k
Connections:
- removed net N$38: IC3.-IN, R31.1, R34.1, R49.2, R51.1
- net +12V: now also IC3.-IN, R31.1, R34.1, R49.2; no longer R51.2
Changed lines of the file:
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@@
 <part name="P-10" library="supply1" deviceset="-12V" device=""/>
 <part name="P+8" library="supply1" deviceset="+12V" device=""/>
-<part name="R49" library="resistor" deviceset="R-US_" device="0207/7" value="120K"/>
+<part name="R49" library="resistor" deviceset="R-US_" device="0207/7" value="91k"/>
 <part name="GND40" library="supply1" deviceset="GND" device=""/>
 <part name="R50" library="resistor" deviceset="R-US_" device="0207/7" value="10K"/>
-<part name="R51" library="resistor" deviceset="R-US_" device="0207/7" value="10M"/>
 <part name="P+16" library="supply1" deviceset="+12V" device=""/>
 <part name="D1" library="diode" library_urn="urn:adsk.eagle:library:210" deviceset="1N4148" device="DO35-7" package3d_urn="urn:adsk.eagle:package:43339/2" value=""/>
@@
 <attribute name="VALUE" x="97.79" y="95.758" size="1.778" layer="96"/>
 </instance>
-<instance part="R51" gate="G$1" x="142.24" y="121.92" smashed="yes">
-<attribute name="NAME" x="138.43" y="123.4186" size="1.778" layer="95"/>
-<attribute name="VALUE" x="138.43" y="118.618" size="1.778" layer="96"/>
-</instance>
 <instance part="P+16" gate="1" x="149.86" y="129.54" smashed="yes">
 <attribute name="VALUE" x="152.4" y="129.54" size="1.778" layer="96"/>
@@
 </segment>
 <segment>
-<pinref part="R51" gate="G$1" pin="2"/>
-<wire x1="147.32" y1="121.92" x2="149.86" y2="121.92" width="0.1524" layer="91"/>
 <pinref part="P+16" gate="1" pin="+12V"/>
 <wire x1="149.86" y1="121.92" x2="149.86" y2="127" width="0.1524" layer="91"/>
+<pinref part="R31" gate="G$1" pin="1"/>
+<wire x1="116.84" y1="129.54" x2="132.08" y2="129.54" width="0.1524" layer="91"/>
+<pinref part="IC3" gate="A" pin="-IN"/>
+<wire x1="129.54" y1="101.6" x2="132.08" y2="101.6" width="0.1524" layer="91"/>
+<wire x1="132.08" y1="101.6" x2="132.08" y2="121.92" width="0.1524" layer="91"/>
+<pinref part="R49" gate="G$1" pin="2"/>
+<wire x1="132.08" y1="121.92" x2="127" y2="121.92" width="0.1524" layer="91"/>
+<pinref part="R34" gate="G$1" pin="1"/>
+<wire x1="134.62" y1="101.6" x2="132.08" y2="101.6" width="0.1524" layer="91"/>
+<wire x1="132.08" y1="129.54" x2="132.08" y2="121.92" width="0.1524" layer="91"/>
+<junction x="132.08" y="121.92"/>
+<junction x="132.08" y="101.6"/>
+<wire x1="149.86" y1="121.92" x2="132.08" y2="121.92" width="0.1524" layer="91"/>
 </segment>
 </net>
@@
 </segment>
 </net>
-<net name="N$38" class="0">
-<segment>
-<pinref part="R31" gate="G$1" pin="1"/>
-<wire x1="116.84" y1="129.54" x2="132.08" y2="129.54" width="0.1524" layer="91"/>
-<pinref part="IC3" gate="A" pin="-IN"/>
-<wire x1="129.54" y1="101.6" x2="132.08" y2="101.6" width="0.1524" layer="91"/>
-<wire x1="132.08" y1="101.6" x2="132.08" y2="121.92" width="0.1524" layer="91"/>
-<pinref part="R49" gate="G$1" pin="2"/>
-<wire x1="132.08" y1="121.92" x2="127" y2="121.92" width="0.1524" layer="91"/>
-<pinref part="R34" gate="G$1" pin="1"/>
-<wire x1="134.62" y1="101.6" x2="132.08" y2="101.6" width="0.1524" layer="91"/>
-<wire x1="132.08" y1="129.54" x2="132.08" y2="121.92" width="0.1524" layer="91"/>
-<junction x="132.08" y="121.92"/>
-<pinref part="R51" gate="G$1" pin="1"/>
-<wire x1="132.08" y1="121.92" x2="137.16" y2="121.92" width="0.1524" layer="91"/>
-<junction x="132.08" y="101.6"/>
-</segment>
-</net>
